File: KiCad/BedLevelingSensor.kicad_pcb (KiCad board)
At the start: 2 copper layers, 4 parts, among them J1 CONN_01X02, U1 ATTINY15-1SC, U2 L9110

Commit message: Schematic
Parts:
- added D1: LED, LEDs:LED_0805, F.Cu at (142.2, 109.9)
- added J2: CONN_01X02, Connectors:GS2, F.Cu at (141.7, 124.7)
- added J3: CONN_01X03, Connectors:GS3, F.Cu at (143.9, 118.0)
- added R2: 10K, Resistors_SMD:R_0603_HandSoldering, F.Cu at (143.5, 121.8)
- added R3: 1K, Resistors_SMD:R_0603_HandSoldering, F.Cu at (143.5, 112.9)
- moved J1 23.3 mm to (137.0, 124.7), turned to 90 degrees
- moved U2 17.7 mm to (138.4, 120.3), turned to 90 degrees
- moved R1 1.28 mm to (137.2, 110.4)
Connections:
- U1 pad 2: IA -> IB
- U1 pad 3: IB -> IA
- U1 pad 6: Net-(U1-Pad6) -> LED
Routing:
- net IB: track 0.00 -> 10.6 mm
- net GND: track 0.00 -> 8.11 mm
- net IA: track 0.00 -> 7.40 mm
- net VCC: track 0.00 -> 4.92 mm
- net Net-(R1-Pad2): track 0.00 -> 2.06 mm
Other:
- board outline added: 12.2 x 17 mm

Commit message: Schematic and PCB
Parts:
- J1: value CONN_01X02 -> SOLENOID
- J2: value CONN_01X02 -> Sensor
- J3: value CONN_01X03 -> Input
- moved J2 18.2 mm to (134.2, 108.1), turned to 270 degrees
- moved R2 15.0 mm to (133.0, 111.1), turned to 90 degrees
- moved J3 11.7 mm to (139.1, 107.3), turned to 270 degrees
- moved R1 5.40 mm to (134.5, 115.1), turned to 270 degrees
- moved J1 4.85 mm to (133.7, 121.2), turned to 0 degrees
- moved R3 1.98 mm to (142.1, 114.3)
- moved U2 1.20 mm to (138.0, 121.4), turned to 0 degrees
- moved U1 1.09 mm to (138.0, 113.3), turned to 90 degrees
- moved D1 0.18 mm to (142.1, 110.0), turned to 270 degrees
Routing:
- net GND: track 8.11 -> 23.0 mm, vias 0 -> 2
- net Net-(J1-Pad1): track 0.00 -> 9.10 mm
- net IB: track 10.6 -> 2.25 mm
- net LED: track 0.00 -> 6.48 mm
- net IA: track 7.40 -> 2.25 mm
- net Net-(J3-Pad3): track 0.00 -> 4.99 mm
- net Net-(J1-Pad2): track 0.00 -> 4.53 mm
- net Net-(J2-Pad1): track 0.00 -> 4.07 mm
- net VCC: track 4.92 -> 7.46 mm, vias 0 -> 2
- net Net-(J2-Pad2): track 0.00 -> 2.21 mm
- net Net-(D1-Pad2): track 0.00 -> 2.12 mm
- added copper zone on B.Cu, net GND
- added copper zone on B.Cu, net VCC
Other:
- board size 12.2 x 17 mm -> 11.2 x 19.7 mm
- net class Default: trace_width 0.25 -> 0.5; via_dia 0.6 -> 1.2; via_drill 0.4 -> 0.8
- net class POWER added: clearance 0.2, trace_width 0.7, via_dia 1.2, via_drill 0.8

Commit message: Schematic/PCB adjust
Parts:
- added C1: 2.2uf, Capacitors_SMD:C_0603_HandSoldering, B.Cu at (139.4, 109.7)
- added C2: 100n, Capacitors_SMD:C_0603_HandSoldering, F.Cu at (131.8, 101.9)
- added J4: Prog?dat, Connectors:GS3, F.Cu at (141.0, 105.9)
- added J5: Prog?pwr, Connectors:GS3, F.Cu at (135.1, 111.3)
- J1, J2, R2, U2: moved to B.Cu
- moved J1 20.7 mm to (140.5, 101.6)
- moved U2 15.4 mm to (135.6, 106.2)
- moved R1 9.04 mm to (131.8, 106.4)
- moved J3 7.55 mm to (135.6, 100.6), turned to 90 degrees
- moved U1 7.51 mm to (135.6, 106.2)
- moved J2 7.11 mm to (131.3, 101.6), turned to 180 degrees
- moved R3 5.43 mm to (140.2, 109.2), turned to 180 degrees
- moved R2 4.90 mm to (131.6, 106.4)
- moved D1 2.39 mm to (140.0, 111.0), turned to 0 degrees
Connections:
- net Net-(J2-Pad1) renamed SCK
- net Net-(J3-Pad3) renamed MOSI
- net Net-(R1-Pad2) renamed RST
Routing:
- net VCC: track 7.46 -> 28.9 mm, vias 2 -> 3
- net SCK: track 4.07 -> 15.9 mm, vias 0 -> 3
- net Net-(J1-Pad1): track 9.10 -> 3.31 mm
- net GND: track 23.0 -> 17.4 mm, vias 2 -> 1
- net Net-(J1-Pad2): track 4.53 -> 9.29 mm
- net RST: track 1.72 -> 5.44 mm
- net LED: track 6.48 -> 9.36 mm
- net MOSI: track 4.99 -> 7.76 mm
- net IB: track 2.25 -> 3.44 mm, vias 0 -> 1
- net IA: track 2.25 -> 3.44 mm, vias 0 -> 1
- net Net-(J2-Pad2): track 2.21 -> 3.14 mm
- net (no net): track 0.00 -> 0.51 mm, vias 0 -> 1
- added copper zone on F.Cu, net GND
- removed copper zone on B.Cu, net VCC
Other:
- board size 11.2 x 19.7 mm -> 12.7 x 12.7 mm
- net class Default: trace_width 0.5 -> 0.3; via_dia 1.2 -> 0.6; via_drill 0.8 -> 0.4
- net class POWER: trace_width 0.7 -> 0.6; via_dia 1.2 -> 0.8; via_drill 0.8 -> 0.5
- rule pad_to_mask_clearance: 0.2 -> 0
- board text added: "Coil"
- board text added: "G"
- board text added: "PWM"
- board text added: "RST"
- board text added: "SCK"
- board text added: "SI"
- board text added: "SO"
- board text added: "Sense"

Commit message: minor pcb asjust
Parts:
- U1: footprint Housings_SOIC:SOIC-8_3.9x4.9mm_Pitch1.27mm -> SMD_Packages:SOIC-8-N
- turned U1 to 0 degrees
Changed lines of the file:
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@@
     (links 29)
     (no_connects 2)
-    (area 129.489999 99.517999 142.290001 112.318001)
+    (area 117.118001 92.804 143.845 114.027)
     (thickness 1.6)
     (drawings 18)
@@
     )
   )
-  (module Housings_SOIC:SOIC-8_3.9x4.9mm_Pitch1.27mm (layer F.Cu)
-    (at 135.636 106.172 90)
-    (descr "8-Lead Plastic Small Outline (SN) - Narrow, 3.90 mm Body [SOIC] (see Microchip Packaging Specification 00000049BS.pdf)")
-    (tags "SOIC 1.27")
-    (attr smd)
-    (fp_text reference U1 (at 0 0 90) (layer F.SilkS)
-      (effects (font (size 1 1) (thickness 0.15)))
-    )
-    (fp_text value ATTINY15-1SC (at 0 3.5 90) (layer F.Fab)
-      (effects (font (size 1 1) (thickness 0.15)))
-    )
-    (fp_text user %R (at 0 0 90) (layer F.Fab)
-      (effects (font (size 1 1) (thickness 0.15)))
-    )
-    (fp_line (start -0.95 -2.45) (end 1.95 -2.45) (layer F.Fab) (width 0.1))
-    (fp_line (start 1.95 -2.45) (end 1.95 2.45) (layer F.Fab) (width 0.1))
-    (fp_line (start 1.95 2.45) (end -1.95 2.45) (layer F.Fab) (width 0.1))
-    (fp_line (start -1.95 2.45) (end -1.95 -1.45) (layer F.Fab) (width 0.1))
-    (fp_line (start -1.95 -1.45) (end -0.95 -2.45) (layer F.Fab) (width 0.1))
-    (fp_line (start -3.73 -2.7) (end -3.73 2.7) (layer F.CrtYd) (width 0.05))
-    (fp_line (start 3.73 -2.7) (end 3.73 2.7) (layer F.CrtYd) (width 0.05))
-    (fp_line (start -3.73 -2.7) (end 3.73 -2.7) (layer F.CrtYd) (width 0.05))
-    (fp_line (start -3.73 2.7) (end 3.73 2.7) (layer F.CrtYd) (width 0.05))
-    (fp_line (start -2.075 -2.575) (end -2.075 -2.525) (layer F.SilkS) (width 0.15))
-    (fp_line (start 2.075 -2.575) (end 2.075 -2.43) (layer F.SilkS) (width 0.15))
-    (fp_line (start 2.075 2.575) (end 2.075 2.43) (layer F.SilkS) (width 0.15))
-    (fp_line (start -2.075 2.575) (end -2.075 2.43) (layer F.SilkS) (width 0.15))
-    (fp_line (start -2.075 -2.575) (end 2.075 -2.575) (layer F.SilkS) (width 0.15))
-    (fp_line (start -2.075 2.575) (end 2.075 2.575) (layer F.SilkS) (width 0.15))
-    (fp_line (start -2.075 -2.525) (end -3.475 -2.525) (layer F.SilkS) (width 0.15))
-    (pad 1 smd rect (at -2.7 -1.905 90) (size 1.55 0.6) (layers F.Cu F.Paste F.Mask)
-      (net 12 RST))
-    (pad 2 smd rect (at -2.7 -0.635 90) (size 1.55 0.6) (layers F.Cu F.Paste F.Mask)
-      (net 8 IB))
-    (pad 3 smd rect (at -2.7 0.635 90) (size 1.55 0.6) (layers F.Cu F.Paste F.Mask)
-      (net 9 IA))
-    (pad 4 smd rect (at -2.7 1.905 90) (size 1.55 0.6) (layers F.Cu F.Paste F.Mask)
-      (net 2 GND))
-    (pad 5 smd rect (at 2.7 1.905 90) (size 1.55 0.6) (layers F.Cu F.Paste F.Mask)
-      (net 11 MOSI))
-    (pad 6 smd rect (at 2.7 0.635 90) (size 1.55 0.6) (layers F.Cu F.Paste F.Mask)
-      (net 7 LED))
-    (pad 7 smd rect (at 2.7 -0.635 90) (size 1.55 0.6) (layers F.Cu F.Paste F.Mask)
-      (net 10 SCK))
-    (pad 8 smd rect (at 2.7 -1.905 90) (size 1.55 0.6) (layers F.Cu F.Paste F.Mask)
-      (net 6 VCC))
-    (model Housings_SOIC.3dshapes/SOIC-8_3.9x4.9mm_Pitch1.27mm.wrl
-      (at (xyz 0 0 0))
-      (scale (xyz 1 1 1))
-      (rotate (xyz 0 0 0))
-    )
-  )
   (module SMD_Packages:SOIC-8-N (layer B.Cu)
     (at 135.636 106.172)
@@
       (at (xyz 0 0 0))
       (scale (xyz 1 1 1))
+      (rotate (xyz 0 0 0))
+    )
+  )
+  (module SMD_Packages:SOIC-8-N (layer F.Cu)
+    (at 135.636 106.172)
+    (descr "Module Narrow CMS SOJ 8 pins large")
+    (tags "CMS SOJ")
+    (attr smd)
+    (fp_text reference U1 (at 0 -1.27) (layer F.SilkS)
+      (effects (font (size 1 1) (thickness 0.15)))
+    )
+    (fp_text value ATTINY15-1SC (at 0 1.27) (layer F.Fab)
+      (effects (font (size 1 1) (thickness 0.15)))
+    )
+    (fp_line (start -2.54 -2.286) (end 2.54 -2.286) (layer F.SilkS) (width 0.15))
+    (fp_line (start 2.54 -2.286) (end 2.54 2.286) (layer F.SilkS) (width 0.15))
+    (fp_line (start 2.54 2.286) (end -2.54 2.286) (layer F.SilkS) (width 0.15))
+    (fp_line (start -2.54 2.286) (end -2.54 -2.286) (layer F.SilkS) (width 0.15))
+    (fp_line (start -2.54 -0.762) (end -2.032 -0.762) (layer F.SilkS) (width 0.15))
+    (fp_line (start -2.032 -0.762) (end -2.032 0.508) (layer F.SilkS) (width 0.15))
+    (fp_line (start -2.032 0.508) (end -2.54 0.508) (layer F.SilkS) (width 0.15))
+    (pad 8 smd rect (at -1.905 -3.175) (size 0.508 1.143) (layers F.Cu F.Paste F.Mask)
+      (net 6 VCC))
+    (pad 7 smd rect (at -0.635 -3.175) (size 0.508 1.143) (layers F.Cu F.Paste F.Mask)
+      (net 10 SCK))
+    (pad 6 smd rect (at 0.635 -3.175) (size 0.508 1.143) (layers F.Cu F.Paste F.Mask)
+      (net 7 LED))
+    (pad 5 smd rect (at 1.905 -3.175) (size 0.508 1.143) (layers F.Cu F.Paste F.Mask)
+      (net 11 MOSI))
+    (pad 4 smd rect (at 1.905 3.175) (size 0.508 1.143) (layers F.Cu F.Paste F.Mask)
+      (net 2 GND))
+    (pad 3 smd rect (at 0.635 3.175) (size 0.508 1.143) (layers F.Cu F.Paste F.Mask)
+      (net 9 IA))
+    (pad 2 smd rect (at -0.635 3.175) (size 0.508 1.143) (layers F.Cu F.Paste F.Mask)
+      (net 8 IB))
+    (pad 1 smd rect (at -1.905 3.175) (size 0.508 1.143) (layers F.Cu F.Paste F.Mask)
+      (net 12 RST))
+    (model SMD_Packages.3dshapes/SOIC-8-N.wrl
+      (at (xyz 0 0 0))
+      (scale (xyz 0.5 0.38 0.5))
       (rotate (xyz 0 0 0))
     )
@@
   (segment (start 131.826 105.326) (end 130.64 105.326) (width 0.6) (layer F.Cu) (net 6))
   (via (at 135.128 111.252) (size 0.8) (drill 0.5) (layers F.Cu B.Cu) (net 6))
-  (segment (start 138.872 111.252) (end 139.446 110.678) (width 0.6) (layer B.Cu) (net 6) (status 800000))
+  (segment (start 138.872 111.252) (end 139.446 110.678) (width 0.6) (layer B.Cu) (net 6))
   (segment (start 133.731 103.472) (end 132.494 103.472) (width 0.6) (layer F.Cu) (net 6))
   (segment (start 132.494 103.472) (end 131.826 102.804) (width 0.6) (layer F.Cu) (net 6))
