File: KiCad/BedLevelingSensor.sch (KiCad schematic (older format))
At the start: 4 parts, among them J1 CONN_01X02, U1 ATTINY15-1SC, U2 L9110

Commit message: Schematic
Parts:
- added D1: LED, LEDs:LED_0805, symbol LED
- added J2: CONN_01X02, Connectors:GS2, symbol CONN_01X02
- added J3: CONN_01X03, Connectors:GS3, symbol CONN_01X03
- added R2: 10K, Resistors_SMD:R_0603_HandSoldering, symbol R
- added R3: 1K, Resistors_SMD:R_0603_HandSoldering, symbol R
Connections:
- net GND: now also D1.1 (K), J3.1 (P1), R2.1
- net IA: now also U1.3 (PB4(ADC3)); no longer U1.2 (PB3(ADC2))
- net IB: now also U1.2 (PB3(ADC2)); no longer U1.3 (PB4(ADC3))
- net VCC: now also J3.2 (P2)
- net at U1.5 (PB0(MOSI/AIN0/AREF)): now also J3.3 (P3)
- net LED: now reaches U1.6 (PB1(MISO/AIN1/OC1A))
- net LED: now also R3.2
- net at U1.7 (PB2(SCK/ADC1/T0/INT0)): now also J2.1 (P1)
- new net: J2.2 (P2), R2.2
- new net: D1.2 (A), R3.1
Changed lines of the file:
@@
 $EndComp
 $Comp
-L GND #PWR5
+L GND #PWR01
 U 1 1 5900F042
 P 5750 4150
-F 0 "#PWR5" H 5750 3900 50  0001 C CNN
+F 0 "#PWR01" H 5750 3900 50  0001 C CNN
 F 1 "GND" H 5750 4000 50  0000 C CNN
 F 2 "" H 5750 4150 50  0001 C CNN
@@
 $EndComp
 $Comp
-L VCC #PWR4
+L VCC #PWR02
 U 1 1 5900F059
 P 5750 3650
-F 0 "#PWR4" H 5750 3500 50  0001 C CNN
+F 0 "#PWR02" H 5750 3500 50  0001 C CNN
 F 1 "VCC" H 5750 3800 50  0000 C CNN
 F 2 "" H 5750 3650 50  0001 C CNN
@@
 $EndComp
 $Comp
-L VCC #PWR1
+L VCC #PWR03
 U 1 1 5900F0E9
 P 3200 3850
-F 0 "#PWR1" H 3200 3700 50  0001 C CNN
+F 0 "#PWR03" H 3200 3700 50  0001 C CNN
 F 1 "VCC" H 3200 4000 50  0000 C CNN
 F 2 "" H 3200 3850 50  0001 C CNN
@@
 $EndComp
 $Comp
-L GND #PWR3
+L GND #PWR04
 U 1 1 5900F614
 P 5500 2550
-F 0 "#PWR3" H 5500 2300 50  0001 C CNN
+F 0 "#PWR04" H 5500 2300 50  0001 C CNN
 F 1 "GND" H 5500 2400 50  0000 C CNN
 F 2 "" H 5500 2550 50  0001 C CNN
@@
 $EndComp
 $Comp
-L GND #PWR6
+L GND #PWR05
 U 1 1 5900F658
 P 5950 1950
-F 0 "#PWR6" H 5950 1700 50  0001 C CNN
+F 0 "#PWR05" H 5950 1700 50  0001 C CNN
 F 1 "GND" H 5950 1800 50  0000 C CNN
 F 2 "" H 5950 1950 50  0001 C CNN
@@
 	5950 1950 5500 1950
 $Comp
-L VCC #PWR2
+L VCC #PWR06
 U 1 1 5900F72C
 P 3600 2150
-F 0 "#PWR2" H 3600 2000 50  0001 C CNN
+F 0 "#PWR06" H 3600 2000 50  0001 C CNN
 F 1 "VCC" H 3600 2300 50  0000 C CNN
 F 2 "" H 3600 2150 50  0001 C CNN
@@
 Wire Wire Line
 	4000 2150 4000 2350
-Text GLabel 3500 3950 0    60   Input ~ 0
+Text GLabel 3650 4050 0    60   Input ~ 0
 IA
 Wire Wire Line
@@
 Wire Wire Line
 	5600 2350 5500 2350
-Text GLabel 3650 4050 0    60   Input ~ 0
+Text GLabel 3500 3950 0    60   Input ~ 0
 IB
 Wire Wire Line
@@
 Wire Wire Line
 	3300 2550 4000 2550
+$Comp
+L CONN_01X02 J2
+U 1 1 59020A74
+P 3100 3300
+F 0 "J2" H 3100 3450 50  0000 C CNN
+F 1 "CONN_01X02" V 3200 3300 50  0000 C CNN
+F 2 "Connectors:GS2" H 3100 3300 50  0001 C CNN
+F 3 "" H 3100 3300 50  0001 C CNN
+	1    3100 3300
+	-1   0    0    1
+$EndComp
+Wire Wire Line
+	3750 3850 3450 3850
+Wire Wire Line
+	3450 3850 3450 3350
+Wire Wire Line
+	3450 3350 3300 3350
+$Comp
+L R R2
+U 1 1 59020CBE
+P 3450 3050
+F 0 "R2" V 3530 3050 50  0000 C CNN
+F 1 "10K" V 3450 3050 50  0000 C CNN
+F 2 "Resistors_SMD:R_0603_HandSoldering" V 3380 3050 50  0001 C CNN
+F 3 "" H 3450 3050 50  0001 C CNN
+	1    3450 3050
+	0    1    1    0
+$EndComp
+Wire Wire Line
+	3300 3250 3300 3050
+$Comp
+L GND #PWR07
+U 1 1 59020D4D
+P 3600 3150
+F 0 "#PWR07" H 3600 2900 50  0001 C CNN
+F 1 "GND" H 3600 3000 50  0000 C CNN
+F 2 "" H 3600 3150 50  0001 C CNN
+F 3 "" H 3600 3150 50  0001 C CNN
+	1    3600 3150
+	1    0    0    -1
+$EndComp
+Wire Wire Line
+	3600 3150 3600 3050
+$Comp
+L CONN_01X03 J3
+U 1 1 59020F14
+P 6200 3100
+F 0 "J3" H 6200 3300 50  0000 C CNN
+F 1 "CONN_01X03" V 6300 3100 50  0000 C CNN
+F 2 "Connectors:GS3" H 6200 3100 50  0001 C CNN
+F 3 "" H 6200 3100 50  0001 C CNN
+	1    6200 3100
+	1    0    0    -1
+$EndComp
+Wire Wire Line
+	6000 3200 3750 3200
+Wire Wire Line
+	3750 3200 3750 3650
+$Comp
+L GND #PWR08
+U 1 1 59021151
+P 5800 2850
+F 0 "#PWR08" H 5800 2600 50  0001 C CNN
+F 1 "GND" H 5800 2700 50  0000 C CNN
+F 2 "" H 5800 2850 50  0001 C CNN
+F 3 "" H 5800 2850 50  0001 C CNN
+	1    5800 2850
+	1    0    0    -1
+$EndComp
+Wire Wire Line
+	5800 2850 6000 2850
+Wire Wire Line
+	6000 2850 6000 3000
+$Comp
+L VCC #PWR09
+U 1 1 59021200
+P 5600 3000
+F 0 "#PWR09" H 5600 2850 50  0001 C CNN
+F 1 "VCC" H 5600 3150 50  0000 C CNN
+F 2 "" H 5600 3000 50  0001 C CNN
+F 3 "" H 5600 3000 50  0001 C CNN
+	1    5600 3000
+	1    0    0    -1
+$EndComp
+Wire Wire Line
+	6000 3100 5600 3100
+Wire Wire Line
+	5600 3100 5600 3000
+Text GLabel 3750 3750 0    60   Input ~ 0
+LED
+$Comp
+L LED D1
+U 1 1 59021665
+P 4550 2950
+F 0 "D1" H 4550 3050 50  0000 C CNN
+F 1 "LED" H 4550 2850 50  0000 C CNN
+F 2 "LEDs:LED_0805" H 4550 2950 50  0001 C CNN
+F 3 "" H 4550 2950 50  0001 C CNN
+	1    4550 2950
+	-1   0    0    1
+$EndComp
+$Comp
+L R R3
+U 1 1 590216DE
+P 4250 2950
+F 0 "R3" V 4330 2950 50  0000 C CNN
+F 1 "1K" V 4250 2950 50  0000 C CNN
+F 2 "Resistors_SMD:R_0603_HandSoldering" V 4180 2950 50  0001 C CNN
+F 3 "" H 4250 2950 50  0001 C CNN
+	1    4250 2950
+	0    1    1    0
+$EndComp
+$Comp
+L GND #PWR010
+U 1 1 59021835
+P 4700 2950
+F 0 "#PWR010" H 4700 2700 50  0001 C CNN
+F 1 "GND" H 4700 2800 50  0000 C CNN
+F 2 "" H 4700 2950 50  0001 C CNN
+F 3 "" H 4700 2950 50  0001 C CNN
+	1    4700 2950
+	1    0    0    -1
+$EndComp
+Text GLabel 4100 2950 0    60   Input ~ 0
+LED
 $EndSCHEMATC

Commit message: Schematic and PCB
Parts:
- J1: value CONN_01X02 -> SOLENOID
- J2: value CONN_01X02 -> Sensor
- J3: value CONN_01X03 -> Input
Changed lines of the file:
@@
 P 3050 2250
 F 0 "J1" H 3050 2400 50  0000 C CNN
-F 1 "CONN_01X02" V 3150 2250 50  0000 C CNN
+F 1 "SOLENOID" V 3150 2250 50  0000 C CNN
 F 2 "Connectors:GS2" H 3050 2250 50  0001 C CNN
 F 3 "" H 3050 2250 50  0001 C CNN
@@
 P 3100 3300
 F 0 "J2" H 3100 3450 50  0000 C CNN
-F 1 "CONN_01X02" V 3200 3300 50  0000 C CNN
+F 1 "Sensor" V 3200 3300 50  0000 C CNN
 F 2 "Connectors:GS2" H 3100 3300 50  0001 C CNN
 F 3 "" H 3100 3300 50  0001 C CNN
@@
 P 6200 3100
 F 0 "J3" H 6200 3300 50  0000 C CNN
-F 1 "CONN_01X03" V 6300 3100 50  0000 C CNN
+F 1 "Input" V 6300 3100 50  0000 C CNN
 F 2 "Connectors:GS3" H 6200 3100 50  0001 C CNN
 F 3 "" H 6200 3100 50  0001 C CNN

Commit message: Schematic/PCB adjust
Parts:
- removed J3: Input, Connectors:GS3, symbol CONN_01X03
- added C1: 2.2uf, Capacitors_SMD:C_0603_HandSoldering, symbol C
- added C2: 100n, Capacitors_SMD:C_0603_HandSoldering, symbol C
- added J3: Inp_Power, Connectors:GS2, symbol CONN_01X02
- added J4: Prog?dat, Connectors:GS3, symbol CONN_01X03
- added J5: Prog?pwr, Connectors:GS3, symbol CONN_01X03
- added J6: Inp_data, Connectors:GS2, symbol CONN_01X02
- R2: value 10K -> 1K
Connections:
- net GND: now also J2.2 (P2), C1.2, C2.2, J3.1 (P1), J5.3 (P3); no longer D1.1 (K), R2.1
- net VCC: now also D1.2 (A), C1.1, C2.1, J3.2 (P2), J5.2 (P2)
- net RST: now reaches R1.2, U1.1 (PB5(~RESET~/ADC0))
- net RST: now also J5.1 (P1)
- net MOSI: now reaches U1.5 (PB0(MOSI/AIN0/AREF))
- net MOSI: now also J4.2 (P2), J6.2 (P2)
- net at J2.1 (P1): now also R2.2; no longer U1.7 (PB2(SCK/ADC1/T0/INT0))
- net at R3.1: now also D1.1 (K); no longer D1.2 (A)
- net LED renamed MISO
- net MISO: now also J4.3 (P3), J6.1 (P1)
- new net SCK: J4.1 (P1), R2.1, U1.7 (PB2(SCK/ADC1/T0/INT0))
Other:
- moved on the sheet: D1, R1, R2

Commit message: adjust attiny footprint
Parts:
- J1, J2: footprint Connectors:GS2 -> Capacitors_SMD:C_1210_HandSoldering
- U1: footprint Housings_SOIC:SOIC-8_3.9x4.9mm_Pitch1.27mm -> SMD_Packages:SOIC-8-N
- U2: footprint SMD_Packages:SOIC-8-N -> Housings_SOIC:SOIC-8_3.9x4.9mm_Pitch1.27mm
Changed lines of the file:
@@
 F 0 "U1" H 3950 4300 50  0000 C CNN
 F 1 "ATTINY15-1SC" H 5400 3500 50  0000 C CNN
-F 2 "Housings_SOIC:SOIC-8_3.9x4.9mm_Pitch1.27mm" H 5350 3900 50  0001 C CIN
+F 2 "SMD_Packages:SOIC-8-N" H 5350 3900 50  0001 C CIN
 F 3 "" H 3950 4250 50  0001 C CNN
 	1    4750 3900
@@
 F 0 "U2" H 4300 2800 60  0000 C CNN
 F 1 "L9110" H 5000 1700 60  0000 C CNN
-F 2 "SMD_Packages:SOIC-8-N" H 3600 3200 60  0001 C CNN
+F 2 "Housings_SOIC:SOIC-8_3.9x4.9mm_Pitch1.27mm" H 3600 3200 60  0001 C CNN
 F 3 "" H 3600 3200 60  0001 C CNN
 	1    4800 2250
@@
 F 0 "J1" H 3050 2400 50  0000 C CNN
 F 1 "SOLENOID" V 3150 2250 50  0000 C CNN
-F 2 "Connectors:GS2" H 3050 2250 50  0001 C CNN
+F 2 "Capacitors_SMD:C_1210_HandSoldering" H 3050 2250 50  0001 C CNN
 F 3 "" H 3050 2250 50  0001 C CNN
 	1    3050 2250
@@
 F 0 "J2" H 3100 3450 50  0000 C CNN
 F 1 "Sensor" V 3200 3300 50  0000 C CNN
-F 2 "Connectors:GS2" H 3100 3300 50  0001 C CNN
+F 2 "Capacitors_SMD:C_1210_HandSoldering" H 3100 3300 50  0001 C CNN
 F 3 "" H 3100 3300 50  0001 C CNN
 	1    3100 3300

Commit message: firmware initial commit
Other:
- note added: "PWM"
Changed lines of the file:
@@
 P 6200 3250
 F 0 "J6" H 6200 3400 50  0000 C CNN
-F 1 "Inp_data" H 6450 3250 50  0000 C CNN
+F 1 "Inp_data" H 6450 3300 50  0000 C CNN
 F 2 "Connectors:GS2" H 6200 3250 50  0001 C CNN
 F 3 "" H 6200 3250 50  0001 C CNN
@@
 Wire Wire Line
 	3600 3050 3300 3050
+Text Notes 6300 3350 0    60   ~ 0
+PWM
 $EndSCHEMATC
